File: RTmFM.kicad_pcb (KiCad board)
At the start: 2 copper layers, 150 x 130 mm, 61 parts, among them J1 Conn_02x04_Odd_Even, J2 Conn_01x04, J3 Conn_02x17_Odd_Even, J4 Conn_02x10_Odd_Even, J5 Micro_SD_Card, J6 Conn_01x02, J8 Conn_01x10, J9 Conn_02x15_Odd_Even, U1 SN75176AP, U10 74LS06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

Commit message: Fixed bus interfacing
Parts:
- added R35: 100R, Resistor_THT:R_Axial_DIN0204_L3.6mm_D1.6mm_P7.62mm_Horizontal, F.Cu at (155.9, 52.3)
- added R36: 1k, Resistor_THT:R_Axial_DIN0204_L3.6mm_D1.6mm_P7.62mm_Horizontal, F.Cu at (143.8, 52.2)
- added R37: 1k, Resistor_THT:R_Axial_DIN0204_L3.6mm_D1.6mm_P7.62mm_Horizontal, F.Cu at (118.1, 69.2)
- added R38: 1k, Resistor_THT:R_Axial_DIN0204_L3.6mm_D1.6mm_P7.62mm_Horizontal, F.Cu at (95.1, 50.2)
- added R39: 1k, Resistor_THT:R_Axial_DIN0204_L3.6mm_D1.6mm_P7.62mm_Horizontal, F.Cu at (105.1, 50.2)
- added R40: 1k, Resistor_THT:R_Axial_DIN0204_L3.6mm_D1.6mm_P7.62mm_Horizontal, F.Cu at (122.8, 50.2)
- added R41: 1k, Resistor_THT:R_Axial_DIN0204_L3.6mm_D1.6mm_P7.62mm_Horizontal, F.Cu at (136.1, 49.2)
- C4: value 10uF -> 10uF/16V
- C8: value 100uF -> 100uF/50V; footprint Capacitor_THT:C_Radial_D8.0mm_H11.5mm_P3.50mm -> Capacitor_THT:CP_Radial_D8.0mm_P3.50mm
- J9: value Conn_02x15_Odd_Even -> Conn_02x15_Odd_Even_JALL
- R10, R11, R12, R13, R6, R7, R8, R9: value 10K -> 10k
- moved C4 21.0 mm to (113.7, 154.1), turned to 90 degrees
- moved C5 16.9 mm to (109.1, 156.1), turned to 90 degrees
- moved J5 13.1 mm to (90.5, 162.7)
Connections:
- R34 pad 1: unconnected-(R34-R1-Pad1) -> /DIRECTION
- R34 pad 13: unconnected-(R34-R12-Pad13) -> /DSEL
- R34 pad 2: unconnected-(R34-R2-Pad2) -> /STEP
- R34 pad 3: unconnected-(R34-R3-Pad3) -> /HEAD1
- R34 pad 4: unconnected-(R34-R4-Pad4) -> /HEAD0
- R34 pad 5: unconnected-(R34-R5-Pad5) -> /WRGATE
- R34 pad 6: unconnected-(R34-R6-Pad6) -> /HEAD2
- R34 pad 7: unconnected-(R34-COM2-Pad7) -> GND
- U2 pad 3: VCC -> /DSEL_INV
Routing:
- net VCC: track 703.8 -> 790.6 mm
- net /DSEL_INV: track 45.5 -> 96.0 mm
- net /SD_DAT3: track 45.2 -> 76.0 mm
- net /SD_DAT2: track 49.7 -> 76.5 mm
- net /SD_DAT0: track 55.9 -> 77.1 mm
- net /SD_CLK: track 60.7 -> 77.0 mm, vias 1 -> 0
- net /SD_CMD: track 62.4 -> 77.3 mm
- net /SD_DAT1: track 63.3 -> 76.8 mm
- net /DSEL: track 109.7 -> 122.6 mm
- net /ocTRACK0: track 61.3 -> 65.5 mm
- net /WDATAP: track 34.1 -> 37.8 mm
- net /ocSEEK_CMPLT: track 63.8 -> 67.2 mm
- net /WDATAN: track 32.9 -> 36.2 mm
- net /WRGATE: track 108.5 -> 105.7 mm
- net /HEAD2: track 77.2 -> 74.6 mm
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Other:
- board text added: "RTmFM MFM Emulator Version 1.2"
- board text added: "Thanks To: aswarmofdeadinsects BackpackVacuum baljemmett cdxxxxdxdrtx ChloeRaccoon cobhc2015 daftpunkle ddopaz FollowX ginja04 HotRocksGirl Jeepin247 Karataus82 matt_inx MB60893 MoKHelix pc_magas rasz_pl RemyKap rfprogrammer rhk77 SeasonedBee SleepyDeveloper spankti spiesofmud StreamElements theOldMaster TokenScandi tradesplatter Tylerhoot vitalkanev Wesley_Nixon Zadster"
- board text removed: "RTmFM MFM Emulator Version 1.1"
- board text removed: "Thanks To: aswarmofdeadinsects BackpackVacuum baljemmett cdxxxxdxdrtx ChloeRaccoon cobhc2015 daftpunkle ddopaz FollowX ginja04 HotRocksGirl Jeepin247 Karataus82 matt_inx MB60893 MoKHelix pc_magas rasz_pl RemDogKap rfprogrammer rhk77 SeasonedBee SleepyDeveloper spankti spiesofmud StreamElements theOldMaster TokenScandi tradesplatter Tylerhoot vitalkanev Wesley_Nixon Zadster"
