File: RTmFM.kicad_sch (KiCad schematic)
At the start: 15 parts, among them J1 Conn_02x04_Odd_Even, U1 74HCT138, U2 74LS153, U3 74LS153, U4 74LS153, U5 74LS153, U6 74HCT151, U7 74HCT244, U8 Pico, U9 74HC04

Commit message: Bus interface
Parts:
- removed R4: 100R, symbol Device:R_Small
- added J2: Conn_01x04, symbol Connector_Generic:Conn_01x04
- added J3: Conn_02x17_Odd_Even, symbol Connector_Generic:Conn_02x17_Odd_Even
- added J4: Conn_02x10_Odd_Even, symbol Connector_Generic:Conn_02x10_Odd_Even
- added R10, R11, R12, R13, R6, R7, R8, R9: 10K, symbol Device:R_Small
- added U10: 74LS06, symbol 74xx:74LS06
- added unit 7 of U9
Connections:
- net DRIVE0: now also J3.26 (Pin_26)
- net DRIVE1: now also J3.28 (Pin_28)
- net DRIVE2: now also J3.30 (Pin_30)
- net DRIVE3: now also J3.32 (Pin_32)
- net DSEL: now also U7.1 (1OE), U9.11
- net GND: now also U1.4 (~{E0}), U2.8 (GND), U7.10 (GND), U7.19 (2OE), J2.2 (Pin_2), J2.3 (Pin_3), J3.1 (Pin_1), J3.11 (Pin_11), J3.13 (Pin_13), J3.17 (Pin_17), J3.19 (Pin_19), J3.21 (Pin_21), J3.23 (Pin_23), J3.25 (Pin_25), J3.27 (Pin_27), J3.29 (Pin_29), J3.3 (Pin_3), J3.31 (Pin_31), J3.33 (Pin_33), J3.5 (Pin_5), J3.7 (Pin_7), J3.9 (Pin_9), J4.11 (Pin_11), J4.12 (Pin_12), J4.15 (Pin_15), J4.16 (Pin_16), J4.19 (Pin_19), J4.2 (Pin_2), J4.20 (Pin_20), J4.4 (Pin_4), J4.6 (Pin_6), R10.2, R6.2, R7.2, R8.2, R9.2, U10.7 (GND), U9.7 (GND)
- net HEAD0: now also J3.14 (Pin_14)
- net HEAD1: now also J3.18 (Pin_18)
- net HEAD2: now also J3.4 (Pin_4)
- net VCC: now also U7.20 (VCC), J2.1 (Pin_1), R11.1, R12.1, R13.1, U10.14 (VCC), U9.14 (VCC)
- net WRGATE: now also U7.11 (2A3), J3.6 (Pin_6); no longer R5.1
- net pREADY: now reaches U8.21 (GPIO16)
- net pREADY: now also U7.17 (2A0)
- net pINDEX: now reaches U8.22 (GPIO17)
- net pINDEX: now also U7.8 (1A3)
- net pWRITE_FAULT: now reaches U8.24 (GPIO18)
- net pWRITE_FAULT: now also U7.6 (1A2)
- net pTRACK0: now reaches U8.25 (GPIO19)
- net pTRACK0: now also U7.4 (1A1)
- net pSEEK_CMPLT: now reaches U8.26 (GPIO20)
- net pSEEK_CMPLT: now also U7.2 (1A0)
- net pDIRECTION: now reaches U8.27 (GPIO21)
- net pDIRECTION: now also U7.7 (2Y2), R12.2
- net pSTEP: now reaches U8.29 (GPIO22)
- net pSTEP: now also U7.5 (2Y1), R11.2
- net pWRGATE: now reaches U8.31 (GPIO26_ADC0)
- net pWRGATE: now also R5.1, U7.9 (2Y3), R13.2
- net INDEX: now reaches U7.12 (1Y3)
- net INDEX: now also R9.1, U10.9
- net DIRECTION: now reaches U7.13 (2A2)
- net DIRECTION: now also J3.34 (Pin_34)
- net WRITE_FAULT: now reaches U7.14 (1Y2)
- net WRITE_FAULT: now also R8.1, U10.5
- net STEP: now reaches U7.15 (2A1)
- net STEP: now also J3.24 (Pin_24)
- net TRACK0: now reaches U7.16 (1Y1)
- net TRACK0: now also R7.1, U10.3
- net SEEK_CMPLT: now reaches U7.18 (1Y0)
- net SEEK_CMPLT: now also R6.1, U10.1
- net READY: now reaches U7.3 (2Y0)
- net READY: now also R10.1, U10.11
- net DSEL_INV: now reaches U9.10
- net DSEL_INV: now also U10.13
- net RDATAP: now reaches U6.5 (Z)
- net RDATAP: now also J4.17 (Pin_17)
- net RDATAN: now reaches U6.6 (~{Z})
- net RDATAN: now also J4.18 (Pin_18)
- new net HEAD3: J3.2 (Pin_2)
- new net WDATAN: J4.14 (Pin_14)
- new net WDATAP: J4.13 (Pin_13)
- new net ocDRV_SLCTD: J4.1 (Pin_1), U10.12
- new net ocINDEX: J3.20 (Pin_20), U10.8
- new net ocREADY: J3.22 (Pin_22), U10.10
- new net ocSEEK_CMPLT: J3.8 (Pin_8), U10.2
- new net ocTRACK0: J3.10 (Pin_10), U10.4
- new net ocWRITE_FAULT: J3.12 (Pin_12), U10.6

Commit message: Fixed footprints and started layout
Parts:
- removed R2, R3, R5: 100R, symbol Device:R_Small
- removed U1: 74HCT138, symbol 74xx:74HCT138
- removed U2, U3, U4, U5: 74LS153, symbol 74xx:74LS153
- removed U6: 74HCT151, symbol 74xx:74LS151
- added C1, C2, C3, C5, C6, C7: 100nF, Capacitor_THT:C_Disc_D7.5mm_W2.5mm_P5.00mm, symbol Device:C
- added C4: 10uF, Capacitor_THT:CP_Radial_D5.0mm_P2.50mm, symbol Device:C
- added C8: 100uF, Capacitor_THT:C_Radial_D8.0mm_H11.5mm_P3.50mm, symbol Device:C
- added D1, D2, D3, D4, D5, D6, D7: BAT43, Diode_THT:D_DO-34_SOD68_P7.62mm_Horizontal, symbol Device:D_Schottky
- added J5: Micro_SD_Card, Connector_Card:microSD_HC_Hirose_DM3D-SF, symbol Connector:Micro_SD_Card
- added J6, J7: Conn_01x02, Connector_PinHeader_2.54mm:PinHeader_1x02_P2.54mm_Vertical, symbol Connector_Generic:Conn_01x02
- added R14, R15, R16, R17, R18, R19, R2, R20, R21, R22, R23, R24, R25, R26, R27, R28, R29, R3, R4, R5: R, Resistor_THT:R_Axial_Power_L20.0mm_W6.4mm_P25.40mm, symbol Device:R
- added RN1: 330R, Resistor_THT:R_Array_SIP9, symbol Device:R_Network08
- added U1, U2: SN75176AP, Package_DIP:DIP-8_W7.62mm, symbol Interface_UART:SN75176AP
- J1: footprint (none) -> Connector_PinHeader_2.54mm:PinHeader_2x04_P2.54mm_Vertical
- J2: footprint (none) -> Connector_TE-Connectivity:TE_MATE-N-LOK_350211-1_1x04_P5.08mm_Vertical
- J3: footprint (none) -> CardEdge:PCB Edge 2.54 pitch 34 pin
- J4: footprint (none) -> CardEdge:PCB Edge 2.54 pitch 20 pin
- R1: value 100R -> 470R; footprint (none) -> Resistor_THT:R_Axial_DIN0204_L3.6mm_D1.6mm_P7.62mm_Horizontal
- R10, R11, R12, R13, R6, R7, R8, R9: footprint (none) -> Resistor_THT:R_Axial_DIN0204_L3.6mm_D1.6mm_P7.62mm_Horizontal
- U10: footprint (none) -> Package_DIP:DIP-14_W10.16mm
- U7: footprint (none) -> Package_DIP:DIP-20_W7.62mm
- U8: footprint RPi_Pico:RPi_Pico_SMD_TH -> Module:RaspberryPi_Pico_Common_THT
- U9: value 74HC04 -> 74HCT04; footprint (none) -> Package_DIP:DIP-14_W10.16mm
Connections:
- net DI2 is gone; now on net WDATA: U8.4 (GPIO2)
- net DI3 is gone; now on net HSEL0: U8.5 (GPIO3)
- net DI4 is gone; now on net HSEL1: U8.6 (GPIO4)
- net DI5 is gone; now on net HSEL2: U8.7 (GPIO5)
- net DI6 is gone; now on net pWRGATE: U8.9 (GPIO6)
- net DO0 is gone; now on net DSEL: U8.11 (GPIO8)
- net DO1 is gone; now on net pSTEP: U8.12 (GPIO9)
- net DO2 is gone; now on net pDIRECTION: U8.14 (GPIO10)
- net DO3 is gone; now on net pSEEK_CMPLT: U8.15 (GPIO11)
- net DO4 is gone; now on net pTRACK0: U8.16 (GPIO12)
- net DO5 is gone; now on net pWRITE_FAULT: U8.17 (GPIO13)
- net DO6 is gone; now on net pINDEX: U8.19 (GPIO14)
- net DO7 is gone; now on net pREADY: U8.20 (GPIO15)
- net DIRECTION: now also D7.1 (K)
- net GND: now also C1.2, C2.2, C3.2, C4.2, C5.2, C6.2, C7.2, C8.2, J5.6 (VSS), R14.2, R15.2, R16.2, R17.2, R18.2, R19.2, R2.2, R20.2, R21.2, R22.2, R23.2, R24.2, R25.2, R26.2, R27.2, R28.2, R29.2, R3.2, R4.2, R5.2, U1.2 (~{RE}), U1.3 (DE), U1.5 (GND), U2.5 (GND)
- net HEAD0: now also D2.1 (K)
- net HEAD1: now also D1.1 (K)
- net HEAD2: now also D3.1 (K)
- net HEAD3: now also D4.1 (K)
- net HSEL0: no longer R1.1
- net RDATAN: now also U2.7 (B)
- net RDATAP: now also U2.6 (A)
- net STEP: now also D6.1 (K)
- net VCC: now also J2.4 (Pin_4), R1.1, C1.1, C2.1, C3.1, C6.1, C7.1, C8.1, J7.1 (Pin_1), R20.1, R21.1, R22.1, R23.1, R24.1, R25.1, R26.1, R27.1, R28.1, R29.1, U1.8 (VCC), U2.2 (~{RE}), U2.3 (DE), U2.8 (VCC); no longer J2.1 (Pin_1)
- net VDD: now also U8.36 (3V3), C4.1, C5.1, J5.4 (VDD)
- net WDATA: now also U1.1 (R)
- net WDATAN: now also U1.7 (B)
- net WDATAP: now also U1.6 (A)
- net WRGATE: now also D5.1 (K)
- net pDIRECTION: no longer U8.27 (GPIO21)
- net pINDEX: no longer U8.22 (GPIO17)
- net pREADY: no longer U8.21 (GPIO16)
- net pSEEK_CMPLT: no longer U8.26 (GPIO20)
- net pSTEP: no longer U8.29 (GPIO22)
- net pTRACK0: no longer U8.25 (GPIO19)
- net pWRGATE: no longer U8.31 (GPIO26_ADC0)
- net pWRITE_FAULT: no longer U8.24 (GPIO18)
- net DRV_LED: now reaches U8.34 (GPIO28_ADC2)
- net DRV_LED: now also U9.13
- net at U9.12: now also J6.2 (Pin_2)
- net at R1.2: now also J6.1 (Pin_1)
- net DI0 renamed DOUT
- net DOUT: now also U2.4 (D)
- net DI1: no longer names the net of U8.2 (GPIO1)
- net DI7: no longer names the net of U8.10 (GPIO7)
- new net: D7.2 (A), RN1.2 (R1)
- new net: D4.2 (A), RN1.8 (R7)
- new net: J7.2 (Pin_2), RN1.1 (common)
- new net: D3.2 (A), RN1.7 (R6)
- new net: D2.2 (A), RN1.5 (R4)
- new net: D6.2 (A), RN1.3 (R2)
- new net: D1.2 (A), RN1.4 (R3)
- new net: D5.2 (A), RN1.6 (R5)
- new net +12V: J2.1 (Pin_1), R14.1, R15.1, R16.1, R17.1, R18.1, R19.1, R2.1, R3.1, R4.1, R5.1
- new net SD_CLK: J5.5 (CLK), U8.24 (GPIO18)
- new net SD_CMD: J5.3 (CMD), U8.25 (GPIO19)
- new net SD_DAT0: J5.7 (DAT0), U8.22 (GPIO17)
- new net SD_DAT1: J5.8 (DAT1), U8.21 (GPIO16)
- new net SD_DAT2: J5.1 (DAT2), U8.27 (GPIO21)
- new net SD_DAT3: J5.2 (DAT3/CD), U8.26 (GPIO20)
Other:
- moved on the sheet: J1, J2, J3, J4, R10, R11, R12, R13, R6, R7, R8, R9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

Commit message: Almost finished HW design
Parts:
- removed unit 3 of U9
- U10, U9: footprint Package_DIP:DIP-14_W10.16mm -> Package_DIP:DIP-14_W7.62mm
Connections:
- net RDENA is gone; now on net HSEL2: U9.8
- net HEAD0: now also U9.3; no longer U9.1
- net HEAD1: now also U9.1; no longer U9.3
- net HEAD2: now also U9.9
- net HSEL0: now also U9.4; no longer U9.2
- net HSEL1: now also U9.2; no longer U9.4
- net INDEX: now also U10.5; no longer U10.9
- net TRACK0: now also U10.9; no longer U10.3
- net VCC: now also U8.39 (VSYS)
- net WRGATE: no longer U9.9
- net WRITE_FAULT: now also U10.3; no longer U10.5
- net ocINDEX: now also U10.6; no longer U10.8
- net ocTRACK0: now also U10.8; no longer U10.4
- net ocWRITE_FAULT: now also U10.4; no longer U10.6
Other:
- moved on the sheet: U10B, U10C, U10D, U9A, U9B

Commit message: End of version 1 design
Parts:
- added H1, H2, H3, H4: MountingHole, MountingHole:MountingHole_3.2mm_M3_DIN965_Pad_TopBottom, symbol Mechanical:MountingHole
- added J8: Conn_01x10, Connector_PinHeader_2.54mm:PinHeader_1x10_P2.54mm_Vertical, symbol Connector_Generic:Conn_01x10
- added R30, R31, R32, R33, R34: 100R, Resistor_THT:R_Axial_DIN0204_L3.6mm_D1.6mm_P7.62mm_Horizontal, symbol Device:R_Small
- R14, R15, R16, R17, R18, R19, R2, R20, R21, R22, R23, R24, R25, R26, R27, R28, R29, R3, R4, R5: now not fitted
Connections:
- net DSEL: now also U8.9 (GPIO6); no longer U8.11 (GPIO8)
- net GND: now also J8.1 (Pin_1), J8.7 (Pin_7), J8.9 (Pin_9)
- net HSEL0: now also U8.4 (GPIO2); no longer U8.5 (GPIO3)
- net HSEL1: now also U8.5 (GPIO3); no longer U8.6 (GPIO4)
- net HSEL2: now also U8.6 (GPIO4); no longer U8.7 (GPIO5)
- net VCC: now also J8.10 (Pin_10)
- net VDD: now also J8.8 (Pin_8)
- net WDATA: now also U8.2 (GPIO1); no longer U8.4 (GPIO2)
- net pDIRECTION: now also U8.11 (GPIO8); no longer U8.14 (GPIO10)
- net pINDEX: now also U8.16 (GPIO12); no longer U8.19 (GPIO14)
- net pREADY: now also U8.17 (GPIO13); no longer U8.20 (GPIO15)
- net pSEEK_CMPLT: now also U8.12 (GPIO9); no longer U8.15 (GPIO11)
- net pSTEP: now also U8.10 (GPIO7); no longer U8.12 (GPIO9)
- net pTRACK0: now also U8.14 (GPIO10); no longer U8.16 (GPIO12)
- net pWRGATE: now also U8.7 (GPIO5); no longer U8.9 (GPIO6)
- net pWRITE_FAULT: now also U8.15 (GPIO11); no longer U8.17 (GPIO13)
- net IO2: now reaches U8.29 (GPIO22)
- net IO2: now also R32.1
- net IO3: now reaches U8.31 (GPIO26_ADC0)
- net IO3: now also R33.1
- net IO4: now reaches U8.32 (GPIO27_ADC1)
- net IO4: now also R34.1
- new net: J8.6 (Pin_6), R34.2
- new net: J8.2 (Pin_2), R30.2
- new net: J8.3 (Pin_3), R31.2
- new net: J8.4 (Pin_4), R32.2
- new net: J8.5 (Pin_5), R33.2
- new net IO0: R30.1, U8.20 (GPIO15)
- new net IO1: R31.1, U8.19 (GPIO14)

Commit message: Rework SD interface and add head 4
Parts:
- removed R34: 100R, Resistor_THT:R_Axial_DIN0204_L3.6mm_D1.6mm_P7.62mm_Horizontal, symbol Device:R_Small
- added D8: LED, LED_THT:LED_Rectangular_W5.0mm_H2.0mm_Horizontal_O3.81mm_Z3.0mm, symbol Device:LED
- added unit 4 of U9
- J5: footprint Connector_Card:microSD_HC_Hirose_DM3D-SF -> footprints:503182-1852_MOL
Connections:
- net IO4 is gone; now on net IO3: U8.32 (GPIO27_ADC1)
- net GND: now also J8.4 (Pin_4); no longer U8.42 (GND)
- net HEAD2: now also U9.5; no longer U9.9
- net HEAD3: now also U9.9
- net HSEL2: now also U9.6; no longer U9.8
- net IO1: now also U8.29 (GPIO22); no longer U8.19 (GPIO14)
- net IO2: now also U8.31 (GPIO26_ADC0); no longer U8.29 (GPIO22)
- net IO3: no longer U8.31 (GPIO26_ADC0)
- net SD_CLK: now also U8.21 (GPIO16); no longer U8.24 (GPIO18)
- net SD_CMD: now also U8.22 (GPIO17); no longer U8.25 (GPIO19)
- net SD_DAT0: now also U8.24 (GPIO18); no longer U8.22 (GPIO17)
- net SD_DAT1: now also U8.25 (GPIO19); no longer U8.21 (GPIO16)
- net SD_DAT2: now also U8.26 (GPIO20); no longer U8.27 (GPIO21)
- net SD_DAT3: now also U8.27 (GPIO21); no longer U8.26 (GPIO20)
- net pWRGATE: now also U8.19 (GPIO14); no longer U8.7 (GPIO5)
- net at J8.6 (Pin_6): now also R33.2
- net at D7.2 (A): now also RN1.3 (R2); no longer RN1.2 (R1)
- net at D4.2 (A): now also RN1.9 (R8); no longer RN1.8 (R7)
- net at J6.1 (Pin_1), R1.2: now also D8.2 (A)
- net at D3.2 (A): now also RN1.8 (R7); no longer RN1.7 (R6)
- net at D2.2 (A): now also RN1.6 (R5); no longer RN1.5 (R4)
- net at D6.2 (A): now also RN1.4 (R3); no longer RN1.3 (R2)
- net at D1.2 (A): now also RN1.5 (R4); no longer RN1.4 (R3)
- net at D5.2 (A): now also RN1.7 (R6); no longer RN1.6 (R5)
- net at J6.2 (Pin_2), U9.12: now also D8.1 (K)
- net at R32.2: now also J8.5 (Pin_5); no longer J8.4 (Pin_4)
- new net HSEL3: U8.7 (GPIO5), U9.8
Other:
- moved on the sheet: D1, D2, D3, D4, D5, D6, D7, R32, R33

Commit message: Version 1.1 rework
Parts:
- added J9: Conn_02x15_Odd_Even, Connector_PinHeader_2.54mm:PinHeader_2x15_P2.54mm_Vertical, symbol Connector_Generic:Conn_02x15_Odd_Even
Connections:
- net DOUT: now also J9.17 (Pin_17); no longer U8.1 (GPIO0)
- net DSEL: now also J9.23 (Pin_23); no longer U8.9 (GPIO6)
- net HSEL0: now also J9.25 (Pin_25); no longer U8.4 (GPIO2)
- net HSEL1: now also J9.21 (Pin_21); no longer U8.5 (GPIO3)
- net HSEL2: now also J9.27 (Pin_27); no longer U8.6 (GPIO4)
- net HSEL3: now also J9.29 (Pin_29); no longer U8.7 (GPIO5)
- net WDATA: now also J9.19 (Pin_19); no longer U8.2 (GPIO1)
- net pDIRECTION: now also J9.11 (Pin_11); no longer U8.11 (GPIO8)
- net pINDEX: now also J9.13 (Pin_13); no longer U8.16 (GPIO12)
- net pREADY: now also J9.1 (Pin_1); no longer U8.17 (GPIO13)
- net pSEEK_CMPLT: now also J9.3 (Pin_3); no longer U8.12 (GPIO9)
- net pSTEP: now also J9.7 (Pin_7); no longer U8.10 (GPIO7)
- net pTRACK0: now also J9.5 (Pin_5); no longer U8.14 (GPIO10)
- net pWRGATE: now also J9.15 (Pin_15); no longer U8.19 (GPIO14)
- net pWRITE_FAULT: now also J9.9 (Pin_9); no longer U8.15 (GPIO11)
- new net xDOUT: J9.18 (Pin_18), U8.1 (GPIO0)
- new net xDSEL: J9.24 (Pin_24), U8.9 (GPIO6)
- new net xHSEL0: J9.26 (Pin_26), U8.4 (GPIO2)
- new net xHSEL1: J9.22 (Pin_22), U8.5 (GPIO3)
- new net xHSEL2: J9.28 (Pin_28), U8.6 (GPIO4)
- new net xHSEL3: J9.30 (Pin_30), U8.7 (GPIO5)
- new net xWDATA: J9.20 (Pin_20), U8.2 (GPIO1)
- new net xpDIRECTION: J9.12 (Pin_12), U8.11 (GPIO8)
- new net xpINDEX: J9.14 (Pin_14), U8.16 (GPIO12)
- new net xpREADY: J9.2 (Pin_2), U8.17 (GPIO13)
- new net xpSEEK_CMPLT: J9.4 (Pin_4), U8.12 (GPIO9)
- new net xpSTEP: J9.8 (Pin_8), U8.10 (GPIO7)
- new net xpTRACK0: J9.6 (Pin_6), U8.14 (GPIO10)
- new net xpWRGATE: J9.16 (Pin_16), U8.19 (GPIO14)
- new net xpWRITE_FAULT: J9.10 (Pin_10), U8.15 (GPIO11)

Commit message: Revision 1.1 and working data out
Parts:
- removed D1, D2, D3, D4, D5, D6, D7: BAT43, Diode_THT:D_DO-34_SOD68_P7.62mm_Horizontal, symbol Device:D_Schottky
- removed J7: Conn_01x02, Connector_PinHeader_2.54mm:PinHeader_1x02_P2.54mm_Vertical, symbol Connector_Generic:Conn_01x02
- removed RN1: 330R, Resistor_THT:R_Array_SIP9, symbol Device:R_Network08
- added R34: 220/330, Package_DIP:DIP-14_W7.62mm_Socket, symbol ResistorNetworks:_1
Connections:
- net DIRECTION: now also R34.1 (R1)
- net DRV_LED: now also U8.20 (GPIO15); no longer U8.34 (GPIO28_ADC2)
- net GND: now also R34.7 (COM2)
- net HEAD0: now also R34.4 (R4)
- net HEAD1: now also R34.3 (R3)
- net HEAD2: now also R34.6 (R6)
- net HEAD3: now also R34.9 (R8)
- net IO0: now also U8.29 (GPIO22); no longer U8.20 (GPIO15)
- net IO1: now also U8.31 (GPIO26_ADC0); no longer U8.29 (GPIO22)
- net IO2: now also U8.32 (GPIO27_ADC1); no longer U8.31 (GPIO26_ADC0)
- net IO3: now also U8.34 (GPIO28_ADC2); no longer U8.32 (GPIO27_ADC1)
- net STEP: now also R34.2 (R2)
- net VCC: now also R34.14 (COM1)
- net WRGATE: now also R34.5 (R5)

Commit message: Fixed bus interfacing
Parts:
- added R35: 100R, Resistor_THT:R_Axial_DIN0204_L3.6mm_D1.6mm_P7.62mm_Horizontal, symbol Device:R_Small
- added R36, R37, R38, R39, R40, R41: 1k, Resistor_THT:R_Axial_DIN0204_L3.6mm_D1.6mm_P7.62mm_Horizontal, symbol Device:R_Small
- C4: value 10uF -> 10uF/16V
- C8: value 100uF -> 100uF/50V; footprint Capacitor_THT:C_Radial_D8.0mm_H11.5mm_P3.50mm -> Capacitor_THT:CP_Radial_D8.0mm_P3.50mm
- J9: value Conn_02x15_Odd_Even -> Conn_02x15_Odd_Even_JALL
- R10, R11, R12, R13, R6, R7, R8, R9: value 10K -> 10k
Connections:
- net DSEL: now also R34.13 (R12)
- net DSEL_INV: now also U2.3 (DE)
- net VCC: now also R36.1, R37.1, R38.1, R39.1, R40.1, R41.1; no longer U2.3 (DE)
- net WDATAN: now also R35.1
- net WDATAP: now also R35.2
- net ocDRV_SLCTD: now also R41.2
- net ocINDEX: now also R39.2
- net ocREADY: now also R40.2
- net ocSEEK_CMPLT: now also R36.2
- net ocTRACK0: now also R37.2
- net ocWRITE_FAULT: now also R38.2
